Commit message: rviz2 visualization created

File: urdf/shadow.urdf (robot description, URDF)
Before this commit: robot shadow, 10 links, 9 joints
Links:
- link base_link: geometry collision mesh filename=package://shadow_description/meshes/base_link.stl; visual mesh filename=package://shadow_description/meshes/base_link.stl
- link bpearl: geometry collision mesh filename=package://shadow_description/meshes/bpearl.stl; visual mesh filename=package://shadow_description/meshes/bpearl.stl
- link cap: geometry collision mesh filename=package://shadow_description/meshes/cap.stl; visual mesh filename=package://shadow_description/meshes/cap.stl
- link helios: geometry collision mesh filename=package://shadow_description/meshes/helios.stl; visual mesh filename=package://shadow_description/meshes/helios.stl
- link motor_left: geometry collision mesh filename=package://shadow_description/meshes/motor_front_left.stl; visual mesh filename=package://shadow_description/meshes/motor_front_left.stl
- link motor_right: geometry collision mesh filename=package://shadow_description/meshes/motor_front_right.stl; visual mesh filename=package://shadow_description/meshes/motor_front_right.stl
- link neck: geometry collision mesh filename=package://shadow_description/meshes/neck.stl; visual mesh filename=package://shadow_description/meshes/neck.stl
- link ricoh_theta_z1: geometry collision mesh filename=package://shadow_description/meshes/ricoh_theta_z1.stl; visual mesh filename=package://shadow_description/meshes/ricoh_theta_z1.stl
- link tray: geometry collision mesh filename=package://shadow_description/meshes/tray.stl; visual mesh filename=package://shadow_description/meshes/tray.stl
- link zed_camera_link: geometry collision mesh filename=package://shadow_description/meshes/zed_camera.stl; visual mesh filename=package://shadow_description/meshes/zed_camera.stl
